File: hardware/projects/cs4272-breakout-board/cs4272-breakout-board.sch (EAGLE design)
At the start: 19 parts, among them Q1 24.576M, U1 CS4272

Commit message: Update breakout board
Parts:
- added JP6: APWR, pinhead:PINHD-1X2
- JP1: value (none) -> I2C/SPI
- JP2: value (none) -> AIN; device pinhead:PINHD-1X5 -> pinhead:PINHD-1X6
- JP3: value (none) -> AOUT
- JP4: value (none) -> I2S
- JP5: value (none) -> DPWR; device pinhead:PINHD-1X5 -> pinhead:PINHD-1X3
Connections:
- net !AMUTEC!: now also JP3.1; no longer JP3.3
- net !BMUTEC!: now also JP3.6; no longer JP3.7
- net AINA+: now also JP2.4; no longer JP2.3
- net AINA-: now also JP2.3; no longer JP2.2
- net AINB+: now also JP2.5; no longer JP2.4
- net AINB-: now also JP2.6; no longer JP2.5
- net AOUTA+: now also JP3.3; no longer JP3.4
- net AOUTB+: now also JP3.4; no longer JP3.5
- net AOUTB-: now also JP3.5; no longer JP3.6
- net GND: now also JP3.7, JP4.6, JP6.1; no longer JP3.1, JP4.1
- net LRCK: now also JP4.2; no longer JP4.3
- net MCLK: now also JP4.1; no longer JP4.4
- net SCLK: now also JP4.3; no longer JP4.2
- net SDOUT(M/!S!): now also JP4.4; no longer JP4.6
- net VA: now also JP6.2; no longer JP5.2
- net VCOM: now also JP2.2; no longer JP5.5
- net VD: now also JP5.2; no longer JP5.3
- net VL: now also JP5.3; no longer JP5.4
Other:
- moved on the sheet: JP1, JP3, JP4

Commit message: Update breakout board
Parts:
- added R1, R2, R3, R4, R5, R6, R7, R8: (no value), rcl:R-EU_R0603
- JP1: value I2C/SPI -> I2S; device pinhead:PINHD-1X5 -> pinhead:PINHD-1X6
- JP4: value I2S -> I2C/SPI; device pinhead:PINHD-1X6 -> pinhead:PINHD-1X5
Connections:
- new net N$1: JP4.4, R1.1
- new net N$2: JP4.3, R2.1
- new net N$3: JP4.2, R3.1
- new net N$4: JP1.2, R8.1
- new net N$5: JP1.3, R7.1
- new net N$6: JP1.4, R6.1
- new net N$7: JP1.5, R5.1
- new net N$8: JP1.6, R4.1
- net !AMUTEC!: now also JP3.2; no longer JP3.1
- net !BMUTEC!: now also JP3.7; no longer JP3.6
- net !RST!: now also JP4.5; no longer JP1.5
- net AD0/!CS!(I2S/!LJ!): now also R1.2; no longer JP1.4
- net AOUTA+: now also JP3.4; no longer JP3.3
- net AOUTA-: now also JP3.3; no longer JP3.2
- net AOUTB+: now also JP3.5; no longer JP3.4
- net AOUTB-: now also JP3.6; no longer JP3.5
- net GND: now also JP3.1, JP4.1; no longer JP3.7, JP4.6
- net LRCK: now also R7.2; no longer JP4.2
- net MCLK: now also R8.2; no longer JP4.1
- net SCL/CCLK(M0): now also R3.2; no longer JP1.2
- net SCLK: now also R6.2; no longer JP4.3
- net SDA/CDIN(M1): now also R2.2; no longer JP1.3
- net SDIN: now also R4.2; no longer JP4.5
- net SDOUT(M/!S!): now also R5.2; no longer JP4.4
